File: openlst-hw.kicad_sch (KiCad schematic)
At the start: 85 parts, among them J2 CC Prog/Debug, J3 UART0, J4 UART1, J5 Control Outputs, J6 ANT, J7 PC104-1, J8 PC104-2, U1 LM1117-3.3, U2 CC1110, U3 RFFM6406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

Commit message: CAM: commiting current revision
Parts:
- removed J5: Control Outputs, archive:PinHeader_1x03_P2.54mm_Vertical, symbol openlst-hw:Conn_01x03
- removed R13, R14: 100, archive:R_0603_1608Metric, symbol openlst-hw:R
Connections:
- net +5V: no longer J8.25 (Pin_25), J8.26 (Pin_26)
- net 5V_VIN: now also J8.25 (Pin_25), J8.26 (Pin_26)
Changed lines of the file:
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@@
     (stroke (width 0) (type default) (color 0 0 0 0))
   )
-  (wire (pts (xy 40.4368 244.729) (xy 59.4868 244.729))
-    (stroke (width 0) (type default) (color 0 0 0 0))
-  )
   (wire (pts (xy 341.884 38.5064) (xy 341.884 39.7764))
     (stroke (width 0) (type default) (color 0 0 0 0))
   )
-  (wire (pts (xy 32.8168 249.809) (xy 34.0868 249.809))
-    (stroke (width 0) (type default) (color 0 0 0 0))
-  )
   (wire (pts (xy 185.674 85.4964) (xy 190.754 85.4964))
     (stroke (width 0) (type default) (color 0 0 0 0))
@@
     (stroke (width 0) (type default) (color 0 0 0 0))
   )
+  (wire (pts (xy 62.738 173.482) (xy 62.738 174.4726))
+    (stroke (width 0) (type default) (color 0 0 0 0))
+  )
   (wire (pts (xy 362.204 91.8464) (xy 364.744 91.8464))
     (stroke (width 0) (type default) (color 0 0 0 0))
@@
     (stroke (width 0) (type default) (color 0 0 0 0))
   )
-  (wire (pts (xy 40.4368 247.269) (xy 59.4868 247.269))
-    (stroke (width 0) (type default) (color 0 0 0 0))
-  )
   (wire (pts (xy 228.854 108.3564) (xy 241.554 108.3564))
     (stroke (width 0) (type default) (color 0 0 0 0))
@@
     (stroke (width 0) (type default) (color 0 0 0 0))
   )
-  (wire (pts (xy 34.0868 249.809) (xy 34.0868 251.079))
-    (stroke (width 0) (type default) (color 0 0 0 0))
-  )
   (wire (pts (xy 58.674 151.6126) (xy 70.104 151.6126))
     (stroke (width 0) (type default) (color 0 0 0 0))
@@
     (effects (font (size 1.524 1.524)) (justify left bottom))
   )
-  (label "~{LST_RX_MODE}" (at 44.2468 247.269 0)
-    (effects (font (size 1.524 1.524)) (justify left bottom))
-  )
   (label "UART1_RTS" (at 162.814 82.9564 0)
     (effects (font (size 1.524 1.524)) (justify left bottom))
@@
     (effects (font (size 1.524 1.524)) (justify left bottom))
   )
-  (label "LST_TX_MODE" (at 44.2468 244.729 0)
-    (effects (font (size 1.524 1.524)) (justify left bottom))
-  )
   (label "AN1" (at 394.97 228.9048 0)
     (effects (font (size 1.524 1.524)) (justify left bottom))
@@
     (effects (font (size 1.524 1.524)) (justify left bottom))
   )
+  (global_label "5V_VIN" (shape input) (at 90.932 174.4726 0) (fields_autoplaced)
+    (effects (font (size 1.524 1.524)) (justify left))
+    (property "Intersheet References" "${INTERSHEET_REFS}" (id 0) (at 101.2683 174.5678 0)
+      (effects (font (size 1.524 1.524)) (justify left) hide)
+    )
+  )
+  (global_label "5V_VIN" (shape input) (at 62.738 173.482 90) (fields_autoplaced)
+    (effects (font (size 1.524 1.524)) (justify left))
+    (property "Intersheet References" "${INTERSHEET_REFS}" (id 0) (at 62.8332 163.1457 90)
+      (effects (font (size 1.524 1.524)) (justify left) hide)
+    )
+  )
   (global_label "5V_VIN" (shape input) (at 238.1504 221.234 180) (fields_autoplaced)
     (effects (font (size 1.524 1.524)) (justify right))
@@
     (pin "1")
   )
-  (symbol (lib_id "openlst-hw:Conn_01x03") (at 27.7368 247.269 180) (unit 1)
-    (in_bom yes) (on_board yes)
-    (property "Reference" "J5" (id 0) (at 27.7368 252.349 0))
-    (property "Value" "Control Outputs" (id 1) (at 27.7368 242.189 0))
-    (property "Footprint" "archive:PinHeader_1x03_P2.54mm_Vertical" (id 2) (at 27.7368 247.269 0)
-      (effects (font (size 1.27 1.27)) hide)
-    )
-    (property "Datasheet" "" (id 3) (at 27.7368 247.269 0)
-      (effects (font (size 1.27 1.27)) hide)
-    )
-    (pin "1")
-    (pin "2")
-    (pin "3")
-  )
-  (symbol (lib_id "openlst-hw:GND") (at 34.0868 251.079 0) (unit 1)
-    (in_bom yes) (on_board yes)
-    (property "Reference" "#PWR054" (id 0) (at 34.0868 257.429 0)
-      (effects (font (size 1.27 1.27)) hide)
-    )
-    (property "Value" "GND" (id 1) (at 34.0868 254.889 0))
-    (property "Footprint" "" (id 2) (at 34.0868 251.079 0)
-      (effects (font (size 1.27 1.27)) hide)
-    )
-    (property "Datasheet" "" (id 3) (at 34.0868 251.079 0)
-      (effects (font (size 1.27 1.27)) hide)
-    )
-    (pin "1")
-  )
-  (symbol (lib_id "openlst-hw:R") (at 36.6268 247.269 270) (unit 1)
-    (in_bom yes) (on_board yes)
-    (property "Reference" "R14" (id 0) (at 41.7068 248.539 90))
-    (property "Value" "100" (id 1) (at 36.6268 247.269 90))
-    (property "Footprint" "archive:R_0603_1608Metric" (id 2) (at 36.6268 245.491 90)
-      (effects (font (size 1.27 1.27)) hide)
-    )
-    (property "Datasheet" "http://www.yageo.com/NewPortal/yageodocoutput?fileName=/pdf/R-Chip/PYu-AC_51_RoHS_L_6.pdf" (id 3) (at 36.6268 247.269 0)
-      (effects (font (size 1.27 1.27)) hide)
-    )
-    (property "Manuf" "Yageo" (id 4) (at 44.2468 248.539 0)
-      (effects (font (size 1.27 1.27)) hide)
-    )
-    (property "ManufPN" "AC0603FR-07100RL" (id 5) (at 44.2468 248.539 0)
-      (effects (font (size 1.27 1.27)) hide)
-    )
-    (property "Supplier" "Digikey" (id 6) (at 44.2468 248.539 0)
-      (effects (font (size 1.27 1.27)) hide)
-    )
-    (property "SupplierPN" "YAG3561CT-ND" (id 7) (at 44.2468 248.539 0)
-      (effects (font (size 1.27 1.27)) hide)
-    )
-    (pin "1")
-    (pin "2")
-  )
-  (symbol (lib_id "openlst-hw:R") (at 36.6268 244.729 270) (unit 1)
-    (in_bom yes) (on_board yes)
-    (property "Reference" "R13" (id 0) (at 41.7068 245.999 90))
-    (property "Value" "100" (id 1) (at 36.6268 244.729 90))
-    (property "Footprint" "archive:R_0603_1608Metric" (id 2) (at 36.6268 242.951 90)
-      (effects (font (size 1.27 1.27)) hide)
-    )
-    (property "Datasheet" "http://www.yageo.com/NewPortal/yageodocoutput?fileName=/pdf/R-Chip/PYu-AC_51_RoHS_L_6.pdf" (id 3) (at 36.6268 244.729 0)
-      (effects (font (size 1.27 1.27)) hide)
-    )
-    (property "Manuf" "Yageo" (id 4) (at 44.2468 245.999 0)
-      (effects (font (size 1.27 1.27)) hide)
-    )
-    (property "ManufPN" "AC0603FR-07100RL" (id 5) (at 44.2468 245.999 0)
-      (effects (font (size 1.27 1.27)) hide)
-    )
-    (property "Supplier" "Digikey" (id 6) (at 44.2468 245.999 0)
-      (effects (font (size 1.27 1.27)) hide)
-    )
-    (property "SupplierPN" "YAG3561CT-ND" (id 7) (at 44.2468 245.999 0)
-      (effects (font (size 1.27 1.27)) hide)
-    )
-    (pin "1")
-    (pin "2")
-  )
   (symbol (lib_id "openlst-hw:C_Small") (at 288.8234 226.314 0) (unit 1)
     (in_bom yes) (on_board yes)
@@
     (pin "3")
   )
-  (symbol (lib_id "power:+5V") (at 90.932 174.4726 0) (unit 1)
-    (in_bom yes) (on_board yes) (fields_autoplaced)
-    (property "Reference" "#PWR0102" (id 0) (at 90.932 178.2826 0)
-      (effects (font (size 1.27 1.27)) hide)
-    )
-    (property "Value" "+5V" (id 1) (at 90.932 169.6466 0))
-    (property "Footprint" "" (id 2) (at 90.932 174.4726 0)
-      (effects (font (size 1.27 1.27)) hide)
-    )
-    (property "Datasheet" "" (id 3) (at 90.932 174.4726 0)
-      (effects (font (size 1.27 1.27)) hide)
-    )
-    (pin "1")
-  )
   (symbol (lib_id "openlst-hw:GND") (at 60.452 179.5526 0) (unit 1)
     (in_bom yes) (on_board yes) (fields_autoplaced)
@@
     (pin "1")
   )
-  (symbol (lib_id "power:+5V") (at 62.738 174.4726 0) (unit 1)
-    (in_bom yes) (on_board yes) (fields_autoplaced)
-    (property "Reference" "#PWR0103" (id 0) (at 62.738 178.2826 0)
-      (effects (font (size 1.27 1.27)) hide)
-    )
-    (property "Value" "+5V" (id 1) (at 62.738 169.6466 0))
-    (property "Footprint" "" (id 2) (at 62.738 174.4726 0)
-      (effects (font (size 1.27 1.27)) hide)
-    )
-    (property "Datasheet" "" (id 3) (at 62.738 174.4726 0)
-      (effects (font (size 1.27 1.27)) hide)
-    )
-    (pin "1")
-  )
   (symbol (lib_id "Connector_Generic:Conn_02x26_Odd_Even") (at 37.465 174.4726 0) (unit 1)
     (in_bom yes) (on_board yes) (fields_autoplaced)
@@
       (reference "#PWR053") (unit 1) (value "GND") (footprint "")
     )
-    (path "/00000000-0000-0000-0000-00005b31aa01"
-      (reference "#PWR054") (unit 1) (value "GND") (footprint "")
-    )
     (path "/00000000-0000-0000-0000-00005b33e802"
       (reference "#PWR055") (unit 1) (value "+3.3V") (footprint "")
@@
       (reference "#PWR062") (unit 1) (value "GND") (footprint "")
     )
-    (path "/bb3bc9f2-0752-4e4f-920e-9e54317fb7f3"
-      (reference "#PWR0102") (unit 1) (value "+5V") (footprint "")
-    )
-    (path "/c7e65df5-e5d2-4bf1-9c71-a8d2a20a7060"
-      (reference "#PWR0103") (unit 1) (value "+5V") (footprint "")
-    )
     (path "/4451e3f2-a214-4b95-8700-e70376775ae7"
       (reference "#PWR0104") (unit 1) (value "GND") (footprint "")
@@
       (reference "J4") (unit 1) (value "UART1") (footprint "archive:PinHeader_1x06_P2.54mm_Vertical")
     )
-    (path "/00000000-0000-0000-0000-00005b31a0a4"
-      (reference "J5") (unit 1) (value "Control Outputs") (footprint "archive:PinHeader_1x03_P2.54mm_Vertical")
-    )
     (path "/00000000-0000-0000-0000-00005a9a1fb2"
       (reference "J6") (unit 1) (value "ANT") (footprint "coax:SMA_Amphenol_132134_Vertical")
@@
       (reference "R12") (unit 1) (value "100") (footprint "archive:R_0603_1608Metric")
     )
-    (path "/00000000-0000-0000-0000-00005b31d69e"
-      (reference "R13") (unit 1) (value "100") (footprint "archive:R_0603_1608Metric")
-    )
-    (path "/00000000-0000-0000-0000-00005b31cf02"
-      (reference "R14") (unit 1) (value "100") (footprint "archive:R_0603_1608Metric")
-    )
     (path "/00000000-0000-0000-0000-00005b290219"

Commit message: CAM: updated layout to fix some issues with ground plane arrangement
Other:
- note removed: "Control Output"
Changed lines of the file:
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@@
-    (effects (font (size 1.524 1.524) (thickness 0.3048) bold) (justify left bottom))
-  )
-  (text "Control Output" (at 27.5844 220.345 0)
     (effects (font (size 1.524 1.524) (thickness 0.3048) bold) (justify left bottom))
   )
